Commit message: Imported upstream version '2.0.0' of 'upstream'

File: urdf/bcr_bot.xacro (robot description, xacro)
@@ -37,4 +37,5 @@
     <xacro:arg name="ground_truth_frame" default="map"/>
     <xacro:arg name="sim_gazebo" default="false" />
+    <xacro:arg name="sim_ign" default="false" />
     <xacro:arg name="sim_gz" default="false" />
     <xacro:arg name="odometry_source" default="world" />
@@ -46,9 +47,18 @@
         <xacro:include filename="$(find bcr_bot)/urdf/gazebo.xacro"/>
     </xacro:if>
+    <xacro:if value="$(arg sim_ign)">
+        <xacro:include filename="$(find bcr_bot)/urdf/ign.xacro"/>
+    </xacro:if>
     <xacro:if value="$(arg sim_gz)">
         <xacro:include filename="$(find bcr_bot)/urdf/gz.xacro"/>
     </xacro:if>
     <!-- ................................ BASE LINK .................................. -->
+    <link name="base_footprint"/>
     <link name="base_link"/>
+    <joint name="base_joint" type="fixed">
+        <parent link="base_footprint"/>
+        <child link="base_link"/>
+        <origin xyz="0.0 0 ${chassis_height/2 + traction_wheel_radius}" rpy="0 0 0.0" />
+    </joint>
     <link name="chassis_link">
         <collision>

File: urdf/gz.xacro (robot description, xacro)
@@ -3,13 +3,13 @@
     <!-- ........................... SENSOR PLUGIN ................................... -->
     <gazebo>
-        <plugin filename="ignition-gazebo-sensors-system" name="ignition::gazebo::systems::Sensors">
+        <plugin filename="gz-sim-sensors-system" name="gz::sim::systems::Sensors">
             <render_engine>ogre2</render_engine>
         </plugin>
-        <plugin filename="ignition-gazebo-imu-system" name="ignition::gazebo::systems::Imu">
+        <plugin filename="gz-sim-imu-system" name="gz::sim::systems::Imu">
         </plugin>
-        <plugin filename="ignition-gazebo-joint-state-publisher-system" name="ignition::gazebo::systems::JointStatePublisher">
+        <plugin filename="gz-sim-joint-state-publisher-system" name="gz::sim::systems::JointStatePublisher">
         </plugin>
         <!-- ........................... DIFFERENTIAL DRIVE PLUGIN ................................... -->
-        <plugin filename="ignition-gazebo-diff-drive-system" name="ignition::gazebo::systems::DiffDrive">
+        <plugin filename="gz-sim-diff-drive-system" name="gz::sim::systems::DiffDrive">
             <left_joint>middle_left_wheel_joint</left_joint>
             <right_joint>middle_right_wheel_joint</right_joint>
@@ -23,5 +23,5 @@
             </xacro:if>
             <frame_id>odom</frame_id>
-            <child_frame_id>base_link</child_frame_id>
+            <child_frame_id>base_footprint</child_frame_id>
         </plugin>
     </gazebo>
@@ -29,8 +29,8 @@
     <xacro:if value="${odometry_source == 'world'}">
     <gazebo>
-        <plugin filename="libignition-gazebo6-odometry-publisher-system"
-            name="ignition::gazebo::systems::OdometryPublisher">
+        <plugin filename="libgz-sim-odometry-publisher-system"
+            name="gz::sim::systems::OdometryPublisher">
             <odom_frame>odom</odom_frame>
-            <robot_base_frame>base_link</robot_base_frame>
+            <robot_base_frame>base_footprint</robot_base_frame>
             <odom_topic>$(arg wheel_odom_topic)</odom_topic>
             <tf_topic>/tf</tf_topic>
@@ -46,5 +46,5 @@
                 <topic>scan</topic>
                 <update_rate>${two_d_lidar_update_rate}</update_rate>
-                <ignition_frame_id>two_d_lidar</ignition_frame_id>
+                <gz_frame_id>two_d_lidar</gz_frame_id>
                 <lidar>
                     <scan>
@@ -67,6 +67,6 @@
                     </noise>
                 </lidar>
-                <alwaysOn>1</alwaysOn>
-                <visualize>true</visualize>
+                <always_on>1</always_on>
+                <visualize>false</visualize>
             </sensor>
         </gazebo>
@@ -78,7 +78,7 @@
                 <update_rate>30.0</update_rate>
                 <topic>kinect_camera</topic>
-                <ignition_frame_id>kinect_camera</ignition_frame_id>
-                <camera_info_topic>kinect_camera/camera_info</camera_info_topic>
+                <gz_frame_id>kinect_camera</gz_frame_id>
                 <camera>
+                    <camera_info_topic>kinect_camera/camera_info</camera_info_topic>
                     <horizontal_fov>${radians(camera_horizontal_fov)}</horizontal_fov>
                     <image>
@@ -100,5 +100,5 @@
             <always_on>1</always_on>
             <update_rate>1</update_rate>
-            <ignition_frame_id>imu_frame</ignition_frame_id>
+            <gz_frame_id>imu_frame</gz_frame_id>
             <visualize>true</visualize>
             <topic>imu</topic>
@@ -111,5 +111,5 @@
                 <update_rate>10.0</update_rate>
                 <always_on>true</always_on>
-                <ignition_frame_id>stereo_camera_optical</ignition_frame_id>
+                <gz_frame_id>stereo_camera_optical</gz_frame_id>
                 <pose>0 -0.12 0 0 0 0</pose>
                 <topic>stereo_camera/right/image_raw</topic>
@@ -130,5 +130,5 @@
                 <update_rate>10.0</update_rate>
                 <always_on>true</always_on>
-                <ignition_frame_id>stereo_camera_optical</ignition_frame_id>
+                <gz_frame_id>stereo_camera_optical</gz_frame_id>
                 <camera_info_topic>stereo_camera/left/camera_info</camera_info_topic>
                 <pose>0 0 0 0 0 0</pose>
